File: CADFiles/KiCAD/Observatory/Observatory.kicad_pcb (KiCad board)
At the start: 2 copper layers, 204.4 x 75.8 mm, 43 parts, among them J1 prog. LED, J10 Dio_Jump, J11 nRF Connections, J12 Sulu Header, J13 Dio_AD, J14 RsTx_Dio, J15 RsRx_Dio, J16 JScope Voltage, J17 WaveGen. 1 Mux Config., J18 JScope I+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

Commit message: Clean up
Parts:
- moved J23 17.3 mm to (224.5, 112.9)
- moved J22 17.3 mm to (224.5, 43.8)
- moved J20 1.20 mm to (45.4, 112.9)
Routing:
- net DD_DIN_4: track 82.2 -> 72.8 mm
- net DD_DIN_2: track 68.5 -> 64.7 mm
- net AD_Scope2+: track 223.8 -> 220.7 mm
- net AD_Scope1+: track 230.6 -> 228.5 mm
- net DD_DIN_8: track 79.0 -> 77.9 mm
- net JS_V-: vias 27 -> 22
Other:
- board size 204.4 x 75.8 mm -> 204.4 x 77 mm

Commit message: More labels and footprint change.
Parts:
- added G***: LOGO, 3rdPrty_Footprints:NoCrystal, F.Cu at (70.8, 78.5)
- J3: value Digitial Discovery Connection Center -> Digitial Discovery Connection
- U1: footprint Dev_boards:SuLu_Foot -> 3rdPrty_Footprints:SuLu_Foot
Other:
- board text added: "WEST LAB CAPSTONE SCuM - servotory REV1"
