File: CADFiles/KiCAD/Observatory/Observatory.kicad_sch (KiCad schematic)
At the start: 16 parts, among them J1 prog. LED, J10 Dio_Jump, J11 nRF Connections, J12 Sulu Header, J13 Dio_AD, J14 RsTx_Dio, J15 RsRx_Dio, J16 JScope Voltage, J20 Mounting Hole, J21 Mounting Hole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

Commit message: Clean up
Changed lines of the file:
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@@
 	)
 	(junction
-		(at 38.1 127)
+		(at 43.18 127)
 		(diameter 0)
 		(color 0 0 0 0)
@@
 	(wire
 		(pts
-			(xy 34.29 127) (xy 38.1 127)
+			(xy 40.64 127) (xy 43.18 127)
 		)
 		(stroke
@@
 	(wire
 		(pts
-			(xy 38.1 123.19) (xy 38.1 127)
+			(xy 43.18 123.19) (xy 43.18 127)
 		)
 		(stroke
@@
 	(wire
 		(pts
-			(xy 43.18 123.19) (xy 73.66 123.19)
+			(xy 45.72 123.19) (xy 73.66 123.19)
 		)
 		(stroke
@@
 	(wire
 		(pts
-			(xy 35.56 123.19) (xy 38.1 123.19)
+			(xy 40.64 123.19) (xy 43.18 123.19)
 		)
 		(stroke
@@
 	(wire
 		(pts
-			(xy 38.1 127) (xy 49.53 127)
+			(xy 43.18 127) (xy 49.53 127)
 		)
 		(stroke
@@
 	(wire
 		(pts
-			(xy 43.18 119.38) (xy 43.18 123.19)
+			(xy 45.72 119.38) (xy 45.72 123.19)
 		)
 		(stroke
@@
 	(wire
 		(pts
-			(xy 40.64 119.38) (xy 43.18 119.38)
+			(xy 40.64 119.38) (xy 45.72 119.38)
 		)
 		(stroke
@@
 	(global_label "WaveGen.1 Mux  17"
 		(shape input)
-		(at 35.56 123.19 180)
+		(at 40.64 123.19 180)
 		(fields_autoplaced yes)
 		(effects
@@
 		)
 		(property "Intersheetrefs" "${INTERSHEET_REFS}"
-			(at 13.646 123.19 0)
+			(at 18.726 123.19 0)
 			(effects
 				(font
@@
 	(global_label "Scopes Mux  28"
 		(shape input)
-		(at 34.29 127 180)
+		(at 40.64 127 180)
 		(fields_autoplaced yes)
 		(effects
@@
 		)
 		(property "Intersheetrefs" "${INTERSHEET_REFS}"
-			(at 15.6417 127 0)
+			(at 21.9917 127 0)
 			(effects
 				(font

Commit message: More labels and footprint change.
Parts:
- U1: footprint Dev_boards:SuLu_Foot -> 3rdPrty_Footprints:SuLu_Foot
Changed lines of the file:
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@@
 			)
 		)
-		(property "Footprint" "Dev_boards:SuLu_Foot"
+		(property "Footprint" "3rdPrty_Footprints:SuLu_Foot"
 			(at 104.14 62.23 0)
 			(effects
