File: CADFiles/KiCAD/Observatory/Observatory.kicad_sch (KiCad schematic)
At the start: 21 parts, among them J1 GND/CUT, J10 Dio_Jump, J11 nRF Connections, J12 Sulu Header, J13 Dio_AD, J14 RsTx_Dio, J15 RsRx_Dio, J16 JScope Voltage, J20 Mounting Hole, J21 Mounting Hole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

Commit message: Begin REV 2
Parts:
- removed J13: Dio_AD, Connector_PinHeader_2.54mm:PinHeader_2x16_P2.54mm_Vertical, symbol Connector_Generic:Conn_02x16_Odd_Even
- added SW1, SW2: SW_DIP_x08, Button_Switch_THT:SW_DIP_SPSTx08_Slide_9.78x22.5mm_W7.62mm_P2.54mm, symbol Switch:SW_DIP_x08
Connections:
- net AD_DIO_0: now also SW1.16
- net AD_DIO_1: now also SW1.15
- net AD_DIO_10: now also SW2.14
- net AD_DIO_11: now also SW2.13
- net AD_DIO_12: now also SW2.12
- net AD_DIO_13: now also SW2.11
- net AD_DIO_14: now also SW2.10
- net AD_DIO_15: now also SW2.9
- net AD_DIO_2: now also SW1.14
- net AD_DIO_3: now also SW1.13
- net AD_DIO_4: now also SW1.12
- net AD_DIO_5: now also SW1.11
- net AD_DIO_6: now also SW1.10
- net AD_DIO_7: now also SW1.9
- net AD_DIO_8: now also SW2.16
- net AD_DIO_9: now also SW2.15
- net DD_DIN_0: now also J10.2 (Pin_2), J14.2 (Pin_2), SW1.1; no longer J10.4 (Pin_4), J15.2 (Pin_2)
- net DD_DIN_1: now also J10.4 (Pin_4), J15.2 (Pin_2), SW1.2; no longer J10.2 (Pin_2), J14.2 (Pin_2)
- net DD_DIN_10: now also SW1.6
- net DD_DIN_11: now also SW1.8
- net DD_DIN_12: now also SW2.2
- net DD_DIN_13: now also SW2.4
- net DD_DIN_14: now also SW2.6
- net DD_DIN_15: now also SW2.8
- net DD_DIN_2: now also SW1.5
- net DD_DIN_3: now also SW1.7
- net DD_DIN_4: now also SW2.1
- net DD_DIN_5: now also SW2.3
- net DD_DIN_6: now also SW2.5
- net DD_DIN_7: now also SW2.7
- net DD_DIN_8: now also SW1.3
- net DD_DIN_9: now also SW1.4
- net Scopes Mux  1: now also J10.3 (Pin_3); no longer J10.1 (Pin_1)
- net Scopes Mux  2: now also J10.1 (Pin_1); no longer J10.3 (Pin_3)
Other:
- added sheet PICO (pico.kicad_sch)

Commit message: All nets routed.
Parts:
- added J13: Serial, Connector_PinHeader_2.54mm:PinHeader_1x02_P2.54mm_Vertical, symbol Connector:Conn_01x02_Pin
- SW1, SW2: footprint Button_Switch_THT:SW_DIP_SPSTx08_Slide_9.78x22.5mm_W7.62mm_P2.54mm -> Button_Switch_SMD:SW_DIP_SPSTx08_Slide_6.7x21.88mm_W8.61mm_P2.54mm_LowProfile
Connections:
- net AD_DIO_10: now also SW2.11; no longer SW2.14
- net AD_DIO_11: now also SW2.12; no longer SW2.13
- net AD_DIO_12: now also SW2.13; no longer SW2.12
- net AD_DIO_13: now also SW2.14; no longer SW2.11
- net AD_DIO_14: now also SW2.15; no longer SW2.10
- net AD_DIO_15: now also SW2.16; no longer SW2.9
- net AD_DIO_8: now also SW2.9; no longer SW2.16
- net AD_DIO_9: now also SW2.10; no longer SW2.15
- net Scopes Mux  1: now also J10.1 (Pin_1); no longer J10.3 (Pin_3)
- net Scopes Mux  10: now also J10.17 (Pin_17), U1.11a (GPIO4); no longer J10.19 (Pin_19), U1.12a (GPIO12)
- net Scopes Mux  11: now also J10.15 (Pin_15), U1.10a (GPIO11); no longer J10.21 (Pin_21), U1.13a (GPIO5)
- net Scopes Mux  12: now also J10.13 (Pin_13), U1.9a (GPIO3); no longer J10.23 (Pin_23), U1.14a (GPIO13)
- net Scopes Mux  2: now also J10.3 (Pin_3); no longer J10.1 (Pin_1)
- net Scopes Mux  30: now also J13.2 (Pin_2)
- net Scopes Mux  31: now also J13.1 (Pin_1)
- net Scopes Mux  7: now also J10.23 (Pin_23), U1.14a (GPIO13); no longer J10.13 (Pin_13), U1.9a (GPIO3)
- net Scopes Mux  8: now also J10.21 (Pin_21), U1.13a (GPIO5); no longer J10.15 (Pin_15), U1.10a (GPIO11)
- net Scopes Mux  9: now also J10.19 (Pin_19), U1.12a (GPIO12); no longer J10.17 (Pin_17), U1.11a (GPIO4)

Commit message: AD DC(-) error fixed. Jumpers added for feet grounds and DC supplies
Parts:
- added J26, J27, J28, J29: Jumper, Jumper:SolderJumper-2_P1.3mm_Open_Pad1.0x1.5mm, symbol Connector:Conn_01x02_Pin
- added J30: Jumper, Connector_PinHeader_2.54mm:PinHeader_1x02_P2.54mm_Vertical, symbol Connector:Conn_01x02_Pin
Connections:
- net +5V: now also J30.2 (Pin_2); no longer J12.12 (Pin_12), J16.5 (Pin_5), J9.2 (Pin_2), U1.12c (EXT_BAT)
- net GND: now also J26.1 (Pin_1), J27.1 (Pin_1), J28.1 (Pin_1), J29.2 (Pin_2)
- net at J22.1 (Pin_1): now also J28.2 (Pin_2)
- net at J21.1 (Pin_1): now also J27.2 (Pin_2)
- net at J23.1 (Pin_1): now also J29.1 (Pin_1)
- net at J20.1 (Pin_1): now also J26.2 (Pin_2)
- new net: J12.12 (Pin_12), J16.5 (Pin_5), J30.1 (Pin_1), J9.2 (Pin_2), U1.12c (EXT_BAT)
- no-connect marks 11 -> 7
Other:
- company: (none) -> West Lab
- title: (none) -> SCuM Observatory
- moved on the sheet: J9

Commit message: Fixs: Disconnnect pico Vsys from board. RX/TX pin errors, 3WD_CLK pin.
Connections:
- net GND: now also U1.7b (GND); no longer U1.10b (GND)
- net Scopes Mux  30: now also U1.10b (RsTx); no longer U1.9b (RsTx)
- net Scopes Mux  31: now also U1.9b (RsRx); no longer U1.8b (RsRx)
- net at J11.3 (Pin_3): now also U1.8b (3WB_CLK); no longer U1.7b (HARD_RESET)
Changed lines of the file:
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@@
 	(wire
 		(pts
-			(xy 127 161.29) (xy 127 135.89)
+			(xy 127 135.89) (xy 127 168.91)
 		)
 		(stroke
@@
 	(wire
 		(pts
+			(xy 115.57 161.29) (xy 140.97 161.29)
+		)
+		(stroke
+			(width 0)
+			(type default)
+		)
+	)
+	(wire
+		(pts
 			(xy 88.9 104.14) (xy 46.99 104.14)
 		)
@@
 	(wire
 		(pts
-			(xy 140.97 161.29) (xy 127 161.29)
-		)
-		(stroke
-			(width 0)
-			(type default)
-		)
-	)
-	(wire
-		(pts
 			(xy 245.11 151.13) (xy 229.87 151.13)
 		)
@@
 	(wire
 		(pts
-			(xy 115.57 168.91) (xy 115.57 135.89)
-		)
-		(stroke
-			(width 0)
-			(type default)
-		)
-	)
-	(wire
-		(pts
 			(xy 224.79 83.82) (xy 234.95 83.82)
 		)
@@
 	(wire
 		(pts
+			(xy 115.57 161.29) (xy 115.57 135.89)
+		)
+		(stroke
+			(width 0)
+			(type default)
+		)
+	)
+	(wire
+		(pts
 			(xy 88.9 111.76) (xy 52.07 111.76)
 		)
@@
 	(wire
 		(pts
+			(xy 127 168.91) (xy 140.97 168.91)
+		)
+		(stroke
+			(width 0)
+			(type default)
+		)
+	)
+	(wire
+		(pts
 			(xy 217.17 114.3) (xy 243.84 114.3)
 		)
@@
 	(wire
 		(pts
-			(xy 140.97 168.91) (xy 115.57 168.91)
-		)
-		(stroke
-			(width 0)
-			(type default)
-		)
-	)
-	(wire
-		(pts
 			(xy 224.79 86.36) (xy 233.68 86.36)
 		)
@@
 			"UAAAAAAAAACEuKw4fVsAALBHJI94WwAAAAAAAAAAAAAAAAAAAAAAALIBAAAAAAAAAAAAAAAAAADt"
 			"7OzsTLOpPyQjIyMcHLw/AAAAAAAAAABRAAAAAAAAAFDzCY94WwAAEEskj3hbAAAAAAAAAAAAAAAA"
-			"AAAAAAAAsgEAAA=="
+			"AAAAAAAAsgEAAEIAAAAwAAAAKwAAAGoAAABZAAAARgAAAEwAAABJAAAAYQAAADQAAABKAAAAcgAA"
+			"AGEAAABRAAAAbwAAAHQAAAAyAAAAQQAAAFMAAABVAAAAcwAAADQAAABTAAAAcgAAADEAAAB3AAAA"
+			"TQAAAG4AAABOAAAAUAAAAFoAAABmAAAAdQAAAGcAAAB1AAAATgAAAGcAAAA3AAAAQgAAAEcAAABC"
+			"AAAAZwAAADUAAABZAAAARwAAAHIAAABwAAAAeAAAAG0AAABKAAAAegAAAFoAAAA2AAAAYgAAAHIA"
+			"AABXAAAANgAAAFAAAABzAAAAWAAAAE0AAAA2AAAAagAAAE4AAAAzAAAANQAAAE8AAAB5AAAAOAAA"
+			"AEIAAABlAAAAWgAAAGgAAABxAAAARwAAAE0AAAByAAAAeAAAAGwAAABnAAAAbAAAAFcAAAA3AAAA"
+			"cgAAAGwAAABGAAAAYQAAAE8AAAA4AAAAVAAAAEoAAABjAAAAMwAAAGUAAAA0AAAAYwAAAFAAAABs"
+			"AAAANQAAAGEAAABsAAAAdgAAAFgAAABzAAAAZgAAAC8AAABVAAAAWQAAADkAAAA3AAAAOQAAACsA"
+			"AABUAAAAYwAAADAAAABkAAAATwAAADMAAABDAAAAMwAAAEMAAABFAAAATgAAAEcAAAA1AAAAZAAA"
+			"ADAAAABWAAAAbQAAADAAAAA0AAAAeQAAAC8AAABrAAAAcgAAAFQAAAB3AAAAawAAAEsAAABTAAAA"
+			"MAAAAEoAAABlAAAAMwAAADgAAABxAAAAYgAAAHoAAAB6AAAANwAAAGwAAAB6AAAAUAAAAG0AAAA3"
+			"AAAAaAAAAEUAAABSAAAAbQAAAFkAAAAyAAAAVAAAAHUAAABRAAAAMAAAAGwAAABGAAAAQgAAAHkA"
+			"AAArAAAAOAAAAC8AAABJAAAAeQAAADYAAAArAAAAbQAAAFoAAABlAAAAZQAAAFAAAAA0AAAAMQAA"
+			"AGYAAAB2AAAAcgAAAGgAAABWAAAAMwAAAHoAAAArAAAAeQAAAFMAAAAvAAAANQAAADUAAABTAAAA"
+			"OQAAACsAAAB6AAAANwAAAHYAAAB2AAAAdgAAAGsAAAA5AAAASwAAAFMAAABnAAAAcgAAAFQAAABw"
+			"AAAAdQAAAHEAAABnAAAAbwAAAHoAAABrAAAAVgAAAGcAAABhAAAATQAAAEwAAABmAAAAZwAAADYA"
+			"AAAyAAAANQAAAE0AAABRAAAARgAAAHMAAABYAAAAOQAAADEAAABKAAAAegAAAGYAAAAyAAAATAAA"
+			"ACsAAABQAAAAeAAAAGkAAABaAAAAWAAAAGMAAAAzAAAAagAAAC8AAABJAAAAcAAAAGEAAAAzAAAA"
+			"dAAAAFgAAABOAA=="
 		)
 	)
@@
 			"AAATwNovfVsAAAAAAQAAAAAAYAAAAAAAAAAwAAAAAAAAAGOxgS99WwAAAAAAAAAAAACAIvBIQnYA"
 			"AEA/U5h4WwAAcAIAAAAAAABQAAAAAAAAAFOl2i99WwAAAAAAAAAAAAAAAAAAAAAAAAAAAAAAAAAA"
-			"AAABgAAAAAAAAAAAAAAAAAAAAAAAAAAAMBhTmA=="
+			"AAABgAAAAAAAAAAAAAAAAAAAAAAAAAAAMBhTmAF/AACA2p76AX8AABBIn/oBfwAAzoOb+gF/AADa"
+			"g5v6AX8AAOaDm/oBfwAAUEif+gF/AACQSJ/6AX8AANBIn/oBfwAAEEmf+gF/AABASZ/6AX8AAHBJ"
+			"n/oBfwAAP4Sb+gF/AACgSZ/6AX8AAOBJn/oBfwAAQEqf+gF/AACAS5/6AX8AAMBLn/oBfwAAAEyf"
+			"+gF/AABATJ/6AX8AAIBMn/oBfwAAwEyf+gF/AAAgTZ/6AX8AAFBNn/oBfwAAYE2f+gF/AAAgTp/6"
+			"AX8AAEBOn/oBfwAAgE6f+gF/AADATp/6AX8AAPBOn/oBfwAAME+f+gF/AAAohZv6AX8AAHBPn/oB"
+			"fwAA8Jqe+gF/AABAm576AX8AAKBPn/oBfwAA4E+f+gF/AAAgUJ/6AX8AAEBQn/oBfwAAYFCf+gF/"
+			"AAAwUZ/6AX8AAJ6Fm/oBfwAAkKie+gF/AAAgyZ76AX8AANBRn/oBfwAAAFKf+gF/AAAwUp/6AX8A"
+			"AEBSn/oBfwAAcFKf+gF/AACgUp/6AX8AAPBSn/oBfwAAUFOf+gF/AADAU5/6AX8AADBUn/oBfwAA"
+			"sFSf+gF/AADwVJ/6AX8AAEBVn/oBfwAAoFWf+gF/AAAQVp/6AX8AAIBWn/oBfwAAAFef+gF/AABA"
+			"V5/6AX8AAABYn/oBfwAAUFif+gF/AAAQWZ/6AX8AAGBZn/oBfwAAkFmf+gF/AADAWZ/6AX8AANBZ"
+			"n/oBfwAAAFqf+gF/AAAwWp/6AX8AAEBan/oBfwAAUFqf+gF/AACAWp/6AX8AALBan/oBfwAA4Fqf"
+			"+gF/AAAgW5/6AX8AAFBbn/oBfwAAZIeb+gF/AABwh5v6AX8AAJBbn/oBfwAAoFuf+gF/AADgW5/6"
+			"AX8AADBcn/oBfwAAoFyf+gF/AACwXJ/6AX8AAOBcn/oBfwAAIF2f+gF/AABwXZ/6AX8AAMBdn/oB"
+			"fwAAAF6f+gF/AAAwXp/6AX8AAFBen/oBfwAAgF6f+gF/AADAXp/6AX8AACBfn/oBfwAAYF+f+gF/"
+			"AACQX5/6AX8AAMBfn/oBfwAA8F+f+gF/AAAgYJ/6AX8AAGA3n/oBfwAAAAAAAAAAAAAAAAAAAAAA"
+			"AAAAAAAAAAAAAAAAAAAAAADAHcRBAAAAAMDt5BcCfwAAZQAAAAAAAAAAAAAAAAAAAKEDAAAAAAAA"
+			"MAnPinhiAAAwxYyLeGIAAJD8eA6YmtgDwERVg3hiAADQBykO2KWIA7A6Ug642LEDQDVVg3hiAACw"
+			"yU8O2KWIA5D8eA642LEDADpVg3hiAADQBykOuGevA7A6Ug6YmtgDYD9Vg3hiAACwyU8OuGevA5D8"
+			"eA6YmtgDwERVg3hiAACgcLcOAOFDAuDn0g5AWA=="
 		)
 	)
@@
 			"AAAAAAAAAAAAAAAAAAAAAAAAAAAAAAAAAAAAAAAAAAAAAAAAAAAAAAAAAAAAAAAAAAAAAAAAAAAA"
 			"AAAAAAAAAAAAAAAAAAAAAAAAAAAAAAAAAAAAAAAAAAAAAAAAAAAAAAAAAAAAAAAAAAAAAAAAAAAA"
-			"AAAAAAAAAAAAAAAAAAAAAAAAAAAAAAAAAAAAAAAAAAAAAAAAAAAAAAAAAA=="
+			"AAAAAAAAAAAAAAAAAAAAAAAAAAAAAAAAAAAAAAAAAAAAAAAAAAAAAAAAADAAAAAAAAAAtCBQpX5i"
+			"AAABAAAAAQAAADAAAAB4YgAAAAAAAAAAAAAAAAAAAAAAAMEAAAAAAAAAUCrYgnhiAAAgGz9IAn8A"
+			"AGkAAABjAAAAYQAAAGQAAABfAAAAdwAAAGkAAABuAAAAZAAAAG8AAAB3AAAAXwAAAGQAAABlAAAA"
+			"ZgAAAGEAAAB1AAAAbAAAAHQAAABfAAAAdgAAAGEAAAByAAAAaQAAAGEAAABuAAAAdAAAAAAAAACQ"
+			"AAAAAAAAADAAAAAAAAAAtG1QpX5iAAAAAAAAAAAAAEC4P4F4YgAAAAAAAAAAAAAwUwAAAAAAAHAA"
+			"AAAAAAAAZKRfpX5iAAAAAAAAAAAAAKAyIkkCfwAAAAAAAAAAAADwCrOAeGIAAAAAAAAAAAAAR+MM"
+			"AAAAAAAAAAAAAAAAAAAAAAAAAAAAAAAAAAAAAAAAAAAAAAAAAAAAAAAAAAAAAAAAAAAAAAABAwAA"
+			"AAAAAKAPZYJ4YgAAcIGzinhiAAAgAAAAbwAAAHIAAAAgAAAAaAAAAGkAAABkAAAAZQAAACAAAAB0"
+			"AAAAaAAAAGkAAABzAAAAIAAAAGwAAABhAAAAeQAAAGUAAAByAAAAAAAAAAAAAAAAAAAAcQIAAAAA"
+			"AADQ5RKDeGIAAGAWE4N4YgAAAAAAAAAAAAAAAAAAAAAAAAAAAAAAAAAAAAAAAAAAAACAIIAFEgcE"
+			"AP//AAAQAAAAEAAAAAAAAAAAAAAAAAAAAAAAAAAAAAAAAAAAAAAAAAAAAAAAAAAAAAAAAAAAAAAA"
+			"gEPYgnhiAAAAAAAAAAAAACQAAAACAAAAEAAAABAAAAD/////JAAAAAIAAAABAAAAAQAAACQAAAAC"
+			"AAAAEAAAABAAAAD/////AAAAAAAAAAAAAAAAAAAAAAAAAAAQAAAAAAAAABAAAAD//////////woA"
+			"AABAAAAAQAAAAAAAAAAAAAAAAAAAAAAAAAAAAAAAAAAAAAAAAAAAAAAAAAAAAAAAAAAAAAAAAAAA"
+			"AAAAAAAAAAAAAAAAAAAAAAACAAAAAAAAAAAAAABAQtiCeGIAACBC2IJ4YgAAEELYgnhiAAAAAAAA"
+			"AAAAAAAAAAAAAAAAAAAoAAAAAACRAAAAAAAAAJAaE4N4YgAAoBDYgnhiAAAAAAAAAAAAAAAAAAAA"
+			"AAAAAAAAAAAAAAAAAAAAAAAAAAAAAAAAAAAAAAAAAAAAAAAQRNiCeGIAAGAgE4N4YgAAAAAAAAAA"
+			"AAD4////DAAAAA0AAAAAAAAAAAAAAAAAAAAAAAAAAAAAAGAgE4N4YgAAAAIAAAAAAABAAAAAAAAA"
+			"ANQom6R+YgAAOQAAAAAAAAAg/xKDeGIAAACWWUsCfwAAgAAAAAAAAAAAAA=="
 		)
 	)
