File: CADFiles/KiCAD/Observatory/Joule_Scope.kicad_sch (KiCad schematic)
At the start: 4 parts, among them J18 JScope I+, J19 JScope I-, J6 JScope V+, J7 JScope V-

Commit message: AD DC(-) error fixed. Jumpers added for feet grounds and DC supplies
Other:
- company: (none) -> West Lab
- title: (none) -> SCuM Observatory
Changed lines of the file:
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@@
 	(generator_version "9.0")
 	(paper "A4")
+	(title_block
+		(title "SCuM Observatory")
+		(date "2025-03-21")
+		(rev "2")
+		(company "West Lab")
+	)
 	(text "Digikey Part #s\n\nBNC Connection\n	2057-RF1-01A-D-00-75-M-ND	\nBNC Cables\n	900-0732305281-ND"
 		(exclude_from_sim no)
