File: CADFiles/KiCAD/Observatory/RF_Explorer.kicad_sch (KiCad schematic)
At the start: 0 parts

Commit message: AD DC(-) error fixed. Jumpers added for feet grounds and DC supplies
Other:
- company: (none) -> West Lab
- title: (none) -> SCuM Observatory
Changed lines of the file:
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@@
 	(generator_version "9.0")
 	(paper "A4")
+	(title_block
+		(title "SCuM Observatory")
+		(date "2025-03-21")
+		(rev "2")
+		(company "West Lab")
+	)
 )
