File: CADFiles/KiCAD/Observatory/Digital_Discovery.kicad_sch (KiCad schematic)
At the start: 1 part, among them J3 Digitial Discovery Connection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

Commit message: AD DC(-) error fixed. Jumpers added for feet grounds and DC supplies
Other:
- company: (none) -> West Lab
- title: (none) -> SCuM Observatory
Changed lines of the file:
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@@
 	(generator_version "9.0")
 	(paper "A4")
+	(title_block
+		(title "SCuM Observatory")
+		(date "2025-03-21")
+		(rev "2")
+		(company "West Lab")
+	)
 	(rectangle
 		(start 73.66 38.1)
@@
 			"AABiAAAAUwAAAFMAAAB5AAAAWQAAAG0AAABwAAAATgAAAHcAAABsAAAAMAAAAHAAAABJAAAASgAA"
 			"AEkAAAAzAAAAbAAAAE0AAAB5AAAANwAAADUAAABFAAAALwAAAEQAAABlAAAAVgAAAFEAAABxAAAA"
-			"TQAAAEwAAAB6AAAAcgAAAHkAAABzAAAAagAAAEkAAAArAAAARQAAAFMAAAAyAAAAUAAAAHMAAA=="
-		)
-	)
+			"TQAAAEwAAAB6AAAAcgAAAHkAAABzAAAAagAAAEkAAAArAAAARQAAAFMAAAAyAAAAUAAAAHMAAAAA"
+			"AAAAAAAAADAnAAAAAAAAEAEAAAAAAAAGAAAAAAAAAAAAAADAZLQI4I+xBv///3+BjL0Iobe6BrBe"
+			"E5h4WwAAAAAAANDImwcArOkF////f5HwpAfB0/IFYJ5SlHhbAAAAAAAAQOrDB+CPsQb///9/ARLN"
+			"B6G3ugYQWhiYeFsAAAAAAADgCAAI4I+xBv///3+hMAkIobe6BkBBspp4WwAAAAAAAIAnPAjgj7EG"
+			"////f0FPRQiht7oGAAaymnhbAAAAAAAAYG8jCMCEkQb///9/IZcsCIGsmgYgCk6UeFsAAAAAAADg"
+			"CAAI4I+xBv///3+hMAkIobe6BkBBspp4WwAAAAAAAIAnPAjgj7EG////f0FPRQiht7oGAAaymnhb"
+			"AABRCwAAAAAAAMDdbZh4WwAAwE5umHhbAAAAAAAAAAAAAAAAAAAAAAAAMAAAAAAAAABQAAAAAAAA"
+			"AOfcOy19WwAA4NQemHhbAACA/0eYeFsAAAAAAAAAAAAAaQAAAGMAAABoAAAAZQAAAGwAAAB0AAAA"
+			"LgAAAGQAAABlAAAALwAAAEEBAAAAAAAAcBAUmHhbAACQJhOYeFsAAJA6LpB4WwAAkDoukHhbAAAw"
+			"AAAAAAAAAEAAAAAAAAAAZ9M7LX1bAAAAAAAAAAAAAFAQ0wjwvhsDAAAAAAAAAABdAAAAAAAAANAe"
+			"aph4WwAAcAAAAAAAAACwAAAAAAAAAPjD2ftBdgAAAF4TmAAAAAD///9/eFsAAOvP2gzA5WwGwScJ"
+			"AAAAAADBJwkAAAAAAAH//38AAAAA0CDylHhbAACAfCSZeFsAAJB8JJl4WwAAwHwkmXhbAAAgKg+U"
+			"eFsAADAqD5R4WwAAgCoPlHhbAAAAAAGaeFsAAAAAAAAAAAAAAAAAAAAAAAAAAAAAAAAAAAAAAAAA"
+			"AAAAAAAAAAAAAAAAAAAAAAAAACEAAAAAAAAAMH+ymnhbAACQskSYeFsAAMABAAAAAAAAcAAAAAAA"
+			"AAAH/+QvfVsAAHD9XY54WwAAsGSvj3hbAACgZK+PeFsAADAAAAAvAAAATAAAAEUAAABBAAAARAAA"
+			"AEUAAABEAAAASQAAAE4AAABEAAAAVQAAAEMAAABUAAAATwAAAFIAAABTAAAALgAAAKEGAAAAAAAA"
+			"wN1tmHhbAAAgQG6YeFsAAAAAAAAAAAAAAAAAAAAAAABjAAAAdAAAAG8AAAByAAAAIAAAAEEAAAB4"
+			"AAAAaQAAAGEAAABsAAAAQQEAAAAAAABgNBOYeFsAAFAGE5h4WwAAwGZNmnhbAADAZk2aeFsAADAA"
+			"AAAAAAAAQAAAAAAAAABn0TstfVsAAAAAAAAAAAAAgGfYCCAWIQMAAAAAAAAAAGAAAAAAAAAA0A=="
+		)
+	)
