File: BoardFiles/KiCAD/Observatory/Mux_Config.kicad_sch (KiCad schematic)
At the start: 18 parts, among them J17 WaveGen. 1 Mux Config., J4 Scope 1 Mux Config., J5 Scope 2 Mux Config.

Commit message: REV3 DRC pass
Parts:
- removed J17: WaveGen. 1 Mux Config., Button_Switch_SMD:SW_DIP_SPSTx05_Slide_6.7x14.26mm_W8.61mm_P2.54mm_LowProfile, symbol Connector_Generic:Conn_02x05_Top_Bottom
- removed J4: Scope 1 Mux Config., Button_Switch_SMD:SW_DIP_SPSTx05_Slide_6.7x14.26mm_W8.61mm_P2.54mm_LowProfile, symbol Connector_Generic:Conn_02x05_Top_Bottom
- removed J5: Scope 2 Mux Config., Button_Switch_SMD:SW_DIP_SPSTx05_Slide_6.7x14.26mm_W8.61mm_P2.54mm_LowProfile, symbol Connector_Generic:Conn_02x05_Top_Bottom
- removed R10, R11, R12, R13, R14, R15, R16, R2, R3, R4, R5, R6, R7, R8, R9: R_up, Resistor_SMD:R_0805_2012Metric_Pad1.20x1.40mm_HandSolder, symbol Device:R_US
