File: BoardFiles/KiCAD/Observatory/Joule_Scope.kicad_sch (KiCad schematic)
At the start: 6 parts, among them J1 JScope V+, J25 JScope V-, J30 Conn_Coaxial_Small, J33 Conn_Coaxial_Small, J34 JScope I+, J35 JScope I-

Commit message: REV3.1 done. Labels fixed, reverse polarity protection added. Layout impoved.
Parts:
- removed J1: JScope V+, Connector_PinHeader_2.54mm:PinHeader_1x01_P2.54mm_Vertical, symbol Connector:Conn_01x01_Pin
- removed J25: JScope V-, Connector_PinHeader_2.54mm:PinHeader_1x01_P2.54mm_Vertical, symbol Connector:Conn_01x01_Pin
- removed J34: JScope I+, Connector_PinHeader_2.54mm:PinHeader_1x01_P2.54mm_Vertical, symbol Connector:Conn_01x01_Pin
- removed J35: JScope I-, Connector_PinHeader_2.54mm:PinHeader_1x01_P2.54mm_Vertical, symbol Connector:Conn_01x01_Pin
- added J5: JScope V, Connector_PinHeader_2.54mm:PinHeader_1x02_P2.54mm_Vertical, symbol Connector:Conn_01x02_Pin
- added J6: JScope I, Connector_PinHeader_2.54mm:PinHeader_1x02_P2.54mm_Vertical, symbol Connector:Conn_01x02_Pin
Connections:
- net GND: now also J5.1 (Pin_1)
- net JS_I+: now also J6.2 (Pin_2)
- net JS_I-: now also J6.1 (Pin_1)
- net JS_V+: now also J5.2 (Pin_2)
